File: hardware/main-board/main-board.kicad_pcb (KiCad board)
At the start: 2 copper layers, 144.8 x 78.7 mm, 34 parts, among them J1 DMX_In_Connector, J2 DMX_Out_Connector, J3 PSU_Connector, J4 Display_Connector, J5 Remote_Panel _Connector, J6 S2L_Board_Connector, J7 SD_Card_Connector_1, J8 Buttons_Connector, J9 SD_Card_Connector_2, K1 DPDT Relay, K2 DPDT Relay, U1 DMX Input 5V Isolation, U2 6N136, U3 MAX481E, U4 MAX481E, U5 DMX Output 5V Isolation, U6 6N136, U7 ESP32

Commit message: PCB updates
Correction to motherboard R value, update of buttons PCB to rev B as ordered to go in case with reduced clearance
Parts:
- R4: value 120R -> 4.7k
Changed lines of the file:
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@@
       (effects (font (size 1 1) (thickness 0.15)))
     )
-    (fp_text value 120R (at 5.08 2.37 90) (layer F.Fab)
+    (fp_text value 4.7k (at 5.08 2.37 90) (layer F.Fab)
       (effects (font (size 1 1) (thickness 0.15)))
     )
